Commit message: more things

File: franka_ros/franka_description/robots/hand.xacro (robot description, xacro)
@@ -20,9 +20,4 @@
         </geometry>
       </collision>
-      <inertial>
-        <origin xyz="0 0 0" rpy="0 0 0"/>
-        <mass value="0.68"/>
-        <inertia ixx="0.1" ixy="0.0" ixz="0.0" iyy="0.1" iyz="0.0" izz="0.1"/>
-      </inertial>
     </link>
     <link name="${ns}_leftfinger">
@@ -37,9 +32,4 @@
         </geometry>
       </collision>
-      <inertial>
-        <origin xyz="0 0 0" rpy="0 0 0"/>
-        <mass value="0.01"/>
-        <inertia ixx="0.1" ixy="0.0" ixz="0.0" iyy="0.1" iyz="0.0" izz="0.1"/>
-      </inertial>
     </link>
     <link name="${ns}_rightfinger">
@@ -56,9 +46,4 @@
         </geometry>
       </collision>
-      <inertial>
-        <origin xyz="0 0 0" rpy="0 0 0"/>
-        <mass value="0.01"/>
-        <inertia ixx="0.1" ixy="0.0" ixz="0.0" iyy="0.1" iyz="0.0" izz="0.1"/>
-      </inertial>
     </link>
     <joint name="${ns}_finger_joint1" type="prismatic">

File: franka_ros/franka_description/robots/panda_arm.xacro (robot description, xacro)
@@ -1,8 +1,4 @@
 <?xml version='1.0' encoding='utf-8'?>
 <robot xmlns:xacro="http://www.ros.org/wiki/xacro" name="panda">
-  <xacro:arg name="init_pose_xyz" default="0 0 0"/>
-  <xacro:arg name="init_ori_rpy" default="0 0 0"/>
-  <xacro:property name="init_pose" value="$(arg init_pose_xyz)"/>
-  <xacro:property name="init_ori" value="$(arg init_ori_rpy)"/>
   <xacro:macro name="panda_arm" params="arm_id:='panda' description_pkg:='franka_description' connected_to:='' xyz:='0 0 0' rpy:='0 0 0'">
     <xacro:unless value="${not connected_to}">
@@ -13,12 +9,4 @@
       </joint>
     </xacro:unless>
-    <xacro:property name="joint_damping" value="1.0"/>
-    <link name="world" />
-    <joint name="robot_to_world" type="fixed">
-      <parent link="world" />
-      <child link="${arm_id}_link0" />
-      <origin xyz="${init_pose}" rpy="${init_ori}" />
-      <dynamics damping="${joint_damping}"/>
-    </joint>
     <link name="${arm_id}_link0">
       <visual>
@@ -32,9 +20,4 @@
         </geometry>
       </collision>
-      <inertial>
-        <origin xyz="0 0 0" rpy="0 0 0"/>
-        <mass value="3.06"/>
-        <inertia ixx="0.3" ixy="0.0" ixz="0.0" iyy="0.3" iyz="0.0" izz="0.3"/>
-      </inertial>
     </link>
     <link name="${arm_id}_link1">
@@ -49,9 +32,4 @@
         </geometry>
       </collision>
-      <inertial>
-        <origin xyz="0 0 0" rpy="0 0 0"/>
-        <mass value="2.34"/>
-        <inertia ixx="0.3" ixy="0.0" ixz="0.0" iyy="0.3" iyz="0.0" izz="0.3"/>
-      </inertial>
     </link>
     <joint name="${arm_id}_joint1" type="revolute">
@@ -62,5 +40,4 @@
       <axis xyz="0 0 1"/>
       <limit effort="87" lower="-2.8973" upper="2.8973" velocity="2.1750"/>
-      <dynamics damping="${joint_damping}"/>
     </joint>
     <link name="${arm_id}_link2">
@@ -75,9 +52,4 @@
         </geometry>
       </collision>
-      <inertial>
-        <origin xyz="0 0 0" rpy="0 0 0"/>
-        <mass value="2.36"/>
-        <inertia ixx="0.3" ixy="0.0" ixz="0.0" iyy="0.3" iyz="0.0" izz="0.3"/>
-      </inertial>
     </link>
     <joint name="${arm_id}_joint2" type="revolute">
@@ -88,5 +60,4 @@
       <axis xyz="0 0 1"/>
       <limit effort="87" lower="-1.7628" upper="1.7628" velocity="2.1750"/>
-      <dynamics damping="${joint_damping}"/>
     </joint>
     <link name="${arm_id}_link3">
@@ -101,9 +72,4 @@
         </geometry>
       </collision>
-      <inertial>
-        <origin xyz="0 0 0" rpy="0 0 0"/>
-        <mass value="2.38"/>
-        <inertia ixx="0.3" ixy="0.0" ixz="0.0" iyy="0.3" iyz="0.0" izz="0.3"/>
-      </inertial>
     </link>
     <joint name="${arm_id}_joint3" type="revolute">
@@ -114,5 +80,4 @@
       <axis xyz="0 0 1"/>
       <limit effort="87" lower="-2.8973" upper="2.8973" velocity="2.1750"/>
-      <dynamics damping="${joint_damping}"/>
     </joint>
     <link name="${arm_id}_link4">
@@ -127,9 +92,4 @@
         </geometry>
       </collision>
-      <inertial>
-        <origin xyz="0 0 0" rpy="0 0 0"/>
-        <mass value="2.43"/>
-        <inertia ixx="0.3" ixy="0.0" ixz="0.0" iyy="0.3" iyz="0.0" izz="0.3"/>
-      </inertial>
     </link>
     <joint name="${arm_id}_joint4" type="revolute">
@@ -140,5 +100,4 @@
       <axis xyz="0 0 1"/>
       <limit effort="87" lower="-3.0718" upper="-0.0698" velocity="2.1750"/>
-      <dynamics damping="${joint_damping}"/>
     </joint>
     <link name="${arm_id}_link5">
@@ -153,9 +112,4 @@
         </geometry>
       </collision>
-      <inertial>
-        <origin xyz="0 0 0" rpy="0 0 0"/>
-        <mass value="3.5"/>
-        <inertia ixx="0.3" ixy="0.0" ixz="0.0" iyy="0.3" iyz="0.0" izz="0.3"/>
-      </inertial>
     </link>
     <joint name="${arm_id}_joint5" type="revolute">
@@ -166,5 +120,4 @@
       <axis xyz="0 0 1"/>
       <limit effort="12" lower="-2.8973" upper="2.8973" velocity="2.6100"/>
-      <dynamics damping="${joint_damping}"/>
     </joint>
     <link name="${arm_id}_link6">
@@ -179,9 +132,4 @@
         </geometry>
       </collision>
-      <inertial>
-        <origin xyz="0 0 0" rpy="0 0 0"/>
-        <mass value="1.47"/>
-        <inertia ixx="0.3" ixy="0.0" ixz="0.0" iyy="0.3" iyz="0.0" izz="0.3"/>
-      </inertial>
     </link>
     <joint name="${arm_id}_joint6" type="revolute">
@@ -192,5 +140,4 @@
       <axis xyz="0 0 1"/>
       <limit effort="12" lower="-0.0175" upper="3.7525" velocity="2.6100"/>
-      <dynamics damping="${joint_damping}"/>
     </joint>
     <link name="${arm_id}_link7">
@@ -205,9 +152,4 @@
         </geometry>
       </collision>
-      <inertial>
-        <origin xyz="0 0 0" rpy="0 0 0"/>
-        <mass value="0.45"/>
-        <inertia ixx="0.3" ixy="0.0" ixz="0.0" iyy="0.3" iyz="0.0" izz="0.3"/>
-      </inertial>
     </link>
     <joint name="${arm_id}_joint7" type="revolute">
@@ -218,13 +160,6 @@
       <axis xyz="0 0 1"/>
       <limit effort="12" lower="-2.8973" upper="2.8973" velocity="2.6100"/>
-      <dynamics damping="${joint_damping}"/>
     </joint>
-    <link name="${arm_id}_link8">
-      <inertial>
-        <origin xyz="0 0 0" rpy="0 0 0"/>
-        <mass value="0.0"/>
-        <inertia ixx="0.3" ixy="0.0" ixz="0.0" iyy="0.3" iyz="0.0" izz="0.3"/>
-      </inertial>
-    </link>
+    <link name="${arm_id}_link8"/>
     <joint name="${arm_id}_joint8" type="fixed">
       <origin rpy="0 0 0" xyz="0 0 0.107"/>

File: franka_ros/franka_description/robots/panda_arm_hand.urdf.xacro (robot description, xacro)
@@ -1,16 +1,7 @@
 <?xml version="1.0" encoding="utf-8"?>
 <robot xmlns:xacro="http://www.ros.org/wiki/xacro" name="panda">
-  <xacro:arg name="robot_name" default="panda"/>
-  <xacro:arg name="arm_id" default="panda"/>
-  <xacro:arg name="init_pose_xyz" default="0 0 -1"/>
-  <xacro:include filename="$(find franka_description)/robots/panda_arm.xacro">
-      <!--xacro:arg name="init_pose_xyz" value="${init_pose_xyz}"/-->
-  </xacro:include>
+  <xacro:include filename="$(find franka_description)/robots/panda_arm.xacro"/>
   <xacro:include filename="$(find franka_description)/robots/hand.xacro"/>
-  <xacro:include filename="$(find franka_description)/robots/panda.gazebo.xacro"/>
-  <xacro:include filename="$(find franka_description)/robots/panda.transmission.xacro"/>
   <xacro:panda_arm />
   <xacro:hand ns="panda" rpy="0 0 ${-pi/4}" connected_to="panda_link8"/>
-  <xacro:panda_gazebo robot_name="$(arg arm_id)" />
-  <xacro:panda_transmission robot_name="$(arg arm_id)" />
 </robot>
