Commit message: new dual arm formulation

File: franka_gazebo/robots/hand.gazebo.xacro (robot description, xacro)
@@ -1,22 +1,67 @@
 <?xml version='1.0' encoding='utf-8'?>
 <robot xmlns:xacro="http://www.ros.org/wiki/xacro" name="panda">
-	<gazebo reference="${ns}_hand"/>
-	<gazebo reference="${ns}_leftfinger"/>
-	<gazebo reference="${ns}_rightfinger"/>
-	<transmission name="${ns}_finger_joint1_trans">
+	<gazebo reference="panda_left_hand">
+      <material>Gazebo/Grey</material>
+          <mu1>0.2</mu1>
+          <mu2>0.2</mu2>
+  </gazebo>
+	<gazebo reference="panda_left_leftfinger">
+      <material>Gazebo/Grey</material>
+          <mu1>0.2</mu1>
+          <mu2>0.2</mu2>
+  </gazebo>
+	<gazebo reference="panda_left_rightfinger">
+      <material>Gazebo/Grey</material>
+          <mu1>0.2</mu1>
+          <mu2>0.2</mu2>
+  </gazebo>
+  <gazebo reference="panda_right_hand">
+      <material>Gazebo/Grey</material>
+          <mu1>0.2</mu1>
+          <mu2>0.2</mu2>
+  </gazebo>
+  <gazebo reference="panda_right_leftfinger">
+      <material>Gazebo/Grey</material>
+          <mu1>0.2</mu1>
+          <mu2>0.2</mu2>
+  </gazebo>
+  <gazebo reference="panda_right_rightfinger">
+      <material>Gazebo/Grey</material>
+          <mu1>0.2</mu1>
+          <mu2>0.2</mu2>
+  </gazebo>
+	<transmission name="panda_left_finger_joint1_trans">
     <type>transmission_interface/SimpleTransmission</type>
-    <joint name="${ns}_finger_joint1">
+    <joint name="panda_left_finger_joint1">
       <hardwareInterface>hardware_interface/PositionJointInterface</hardwareInterface>
     </joint>
-    <actuator name="${ns}_finger_joint1_motor">
+    <actuator name="panda_left_finger_joint1_motor">
       <mechanicalReduction>1</mechanicalReduction>
     </actuator>
   </transmission>
-  <transmission name="${ns}_finger_joint2_trans">
+  <transmission name="panda_left_finger_joint2_trans">
     <type>transmission_interface/SimpleTransmission</type>
-    <joint name="${ns}_finger_joint2">
+    <joint name="panda_left_finger_joint2">
       <hardwareInterface>hardware_interface/PositionJointInterface</hardwareInterface>
     </joint>
-    <actuator name="${ns}_finger_joint2_motor">
+    <actuator name="panda_left_finger_joint2_motor">
+      <mechanicalReduction>1</mechanicalReduction>
+    </actuator>
+  </transmission>
+  <transmission name="panda_right_finger_joint1_trans">
+    <type>transmission_interface/SimpleTransmission</type>
+    <joint name="panda_right_finger_joint1">
+      <hardwareInterface>hardware_interface/PositionJointInterface</hardwareInterface>
+    </joint>
+    <actuator name="panda_right_finger_joint1_motor">
+      <mechanicalReduction>1</mechanicalReduction>
+    </actuator>
+  </transmission>
+  <transmission name="panda_right_finger_joint2_trans">
+    <type>transmission_interface/SimpleTransmission</type>
+    <joint name="panda_right_finger_joint2">
+      <hardwareInterface>hardware_interface/PositionJointInterface</hardwareInterface>
+    </joint>
+    <actuator name="panda_right_finger_joint2_motor">
       <mechanicalReduction>1</mechanicalReduction>
     </actuator>

File: franka_gazebo/robots/hand.xacro (robot description, xacro)
@@ -1,5 +1,5 @@
 <?xml version="1.0" encoding="utf-8"?>
 <robot xmlns:xacro="http://www.ros.org/wiki/xacro" name="hand">
-  <xacro:macro name="hand" params="connected_to:='' ns:='' rpy:='0 0 0' xyz:='0 0 0' ">
+  <xacro:macro name="hand" params="connected_to:='' ns:='' rpy:='0 0 0' xyz:='0 0 0' safety_distance:=0">
     <xacro:unless value="${connected_to == ''}">
       <joint name="${ns}_hand_joint" type="fixed">
@@ -9,75 +9,77 @@
       </joint>
     </xacro:unless>
-    <xacro:arg name="gazebo" default="true"/>
-    <xacro:if value="$(arg gazebo)">
-      <!-- Gazebo Tags -->
-      <xacro:include filename="$(find franka_gazebo)/robots/hand.gazebo.xacro"/>
-    </xacro:if>
     <link name="${ns}_hand">
-      <inertial>
-        <mass value="0.73" />
-        <origin xyz="0 0.0015244 0.0275912" rpy="0 0 0" />
-        <inertia ixx="0.00278560230025" ixy="0.0" ixz="0.0" iyy="0.000400033405336" iyz="0.0" izz="0.00256378041832" />
-      </inertial>
       <visual>
-        <origin xyz="${xyz}" rpy="0 0 0"/>
         <geometry>
-          <mesh filename="package://franka_gazebo/meshes/visual/hand.dae"/>
+          <mesh filename="package://franka_description/meshes/visual/hand.dae"/>
         </geometry>
-        <material name="">
-          <color rgba="1 1 1 1"/>
-        </material>
       </visual>
       <collision>
-        <origin xyz="${xyz}" rpy="0 0 0"/>
+        <origin xyz="0 0 0.04" rpy="0 ${pi/2} ${pi/2}"/>
         <geometry>
-          <mesh filename="package://franka_gazebo/meshes/collision/hand.stl"/>
+          <cylinder radius="${0.04+safety_distance}" length="0.1" />
         </geometry>
       </collision>
+      <collision>
+        <origin xyz="0 -0.05 0.04" rpy="0 0 0"/>
+        <geometry>
+          <sphere radius="${0.04+safety_distance}"  />
+        </geometry>
+      </collision>
+      <collision>
+        <origin xyz="0 0.05 0.04" rpy="0 0 0"/>
+        <geometry>
+          <sphere radius="${0.04+safety_distance}"  />
+        </geometry>
+      </collision>
+      <collision>
+        <origin xyz="0 0 0.1" rpy="0 ${pi/2} ${pi/2}"/>
+        <geometry>
+          <cylinder radius="${0.02+safety_distance}" length="0.1" />
+        </geometry>
+      </collision>
+      <collision>
+        <origin xyz="0 -0.05 0.1" rpy="0 0 0"/>
+        <geometry>
+          <sphere radius="${0.02+safety_distance}"  />
+        </geometry>
+      </collision>
+      <collision>
+        <origin xyz="0 0.05 0.1" rpy="0 0 0"/>
+        <geometry>
+          <sphere radius="${0.02+safety_distance}"  />
+        </geometry>
+      </collision>
+      <inertial>
+        <origin xyz="0 0 0" rpy="0 0 0"/>
+        <mass value="0.68"/>
+        <inertia ixx="0.1" ixy="0.0" ixz="0.0" iyy="0.1" iyz="0.0" izz="0.1"/>
+      </inertial>
     </link>
     <link name="${ns}_leftfinger">
+      <visual>
+        <geometry>
+          <mesh filename="package://franka_description/meshes/visual/finger.dae"/>
+        </geometry>
+      </visual>
       <inertial>
-        <mass value="0.1" />
-        <origin xyz="0 0.0145644 0.0227941" rpy="0 0 0" />
-        <inertia ixx="3.01220925051e-05" ixy="0.0" ixz="0.0" iyy="2.95873808038e-05" iyz="0.0" izz="6.95125211657e-06" />
+        <origin xyz="0 0 0" rpy="0 0 0"/>
+        <mass value="0.01"/>
+        <inertia ixx="0.1" ixy="0.0" ixz="0.0" iyy="0.1" iyz="0.0" izz="0.1"/>
       </inertial>
-      <visual>
-        <origin xyz="${xyz}" rpy="0 0 0"/>
-        <geometry>
-          <mesh filename="package://franka_gazebo/meshes/visual/finger.dae"/>
-        </geometry>
-        <material name="">
-          <color rgba="1 1 1 1"/>
-        </material>
-      </visual>
-      <collision>
-        <origin xyz="${xyz}" rpy="0 0 0"/>
-        <geometry>
-          <mesh filename="package://franka_gazebo/meshes/collision/finger.stl"/>
-        </geometry>
-      </collision>
     </link>
     <link name="${ns}_rightfinger">
-      <inertial>
-        <mass value="0.1" />
-        <origin xyz="0 0.0145644 0.0227941" rpy="0 0 ${pi}" />
-        <inertia ixx="3.01220925051e-05" ixy="0.0" ixz="0.0" iyy="2.95873808038e-05" iyz="0.0" izz="6.95125211657e-06" />
-      </inertial>
       <visual>
         <origin xyz="0 0 0" rpy="0 0 ${pi}"/>
         <geometry>
-          <mesh filename="package://franka_gazebo/meshes/visual/finger.dae"/>
+          <mesh filename="package://franka_description/meshes/visual/finger.dae"/>
         </geometry>
-        <material name="">
-          <color rgba="1 1 1 1"/>
-        </material>
       </visual>
-      <collision>
-        <origin xyz="0 0 0" rpy="0 0 ${pi}"/>
-        <geometry>
-          <mesh filename="package://franka_gazebo/meshes/collision/finger.stl"/>
-        </geometry>
-      </collision>
-    </link>
+      <inertial>
+        <origin xyz="0 0 0" rpy="0 0 0"/>
+        <mass value="0.01"/>
+        <inertia ixx="0.1" ixy="0.0" ixz="0.0" iyy="0.1" iyz="0.0" izz="0.1"/>
+      </inertial>
+   </link>
     <joint name="${ns}_finger_joint1" type="prismatic">
       <parent link="${ns}_hand"/>
@@ -85,5 +87,5 @@
       <origin xyz="0 0 0.0584" rpy="0 0 0"/>
       <axis xyz="0 1 0"/>
-      <limit effort="20" lower="-0.001" upper="0.04" velocity="0.3"/>
+      <limit effort="20" lower="0.0" upper="0.04" velocity="0.2"/>
     </joint>
     <joint name="${ns}_finger_joint2" type="prismatic">
@@ -92,5 +94,6 @@
       <origin xyz="0 0 0.0584" rpy="0 0 0"/>
       <axis xyz="0 -1 0"/>
-      <limit effort="20" lower="-0.001" upper="0.04" velocity="0.3"/>
+      <limit effort="20" lower="0.0" upper="0.04" velocity="0.2"/>
+      <mimic joint="${ns}_finger_joint1" />
     </joint>
   </xacro:macro>

File: franka_gazebo/robots/panda_arm.gazebo.xacro (robot description, xacro)
@@ -6,73 +6,217 @@
     </plugin>
   </gazebo>
-	<gazebo reference="${arm_id}_link0"/>
-	<gazebo reference="${arm_id}_link1"/>
-	<gazebo reference="${arm_id}_link2"/>
-	<gazebo reference="${arm_id}_link3"/>
-	<gazebo reference="${arm_id}_link4"/>
-	<gazebo reference="${arm_id}_link5"/>
-	<gazebo reference="${arm_id}_link6"/>
-	<gazebo reference="${arm_id}_link7"/>
-	<gazebo reference="${arm_id}_link8"/>
-	 <transmission name="${arm_id}_joint1_trans">
-    <type>transmission_interface/SimpleTransmission</type>
-    <joint name="${arm_id}_joint1">
-      <hardwareInterface>hardware_interface/PositionJointInterface</hardwareInterface>
-    </joint>
-    <actuator name="${arm_id}_joint1_motor">
-      <mechanicalReduction>1</mechanicalReduction>
-    </actuator>
-  </transmission>
-  <transmission name="${arm_id}_joint2_trans">
-    <type>transmission_interface/SimpleTransmission</type>
-    <joint name="${arm_id}_joint2">
-      <hardwareInterface>hardware_interface/PositionJointInterface</hardwareInterface>
-    </joint>
-    <actuator name="${arm_id}_joint2_motor">
-      <mechanicalReduction>1</mechanicalReduction>
-    </actuator>
-  </transmission>
-  <transmission name="${arm_id}_joint3_trans">
-    <type>transmission_interface/SimpleTransmission</type>
-    <joint name="${arm_id}_joint3">
-      <hardwareInterface>hardware_interface/PositionJointInterface</hardwareInterface>
-    </joint>
-    <actuator name="${arm_id}_joint3_motor">
-      <mechanicalReduction>1</mechanicalReduction>
-    </actuator>
-  </transmission>
-  <transmission name="${arm_id}_joint4_trans">
-    <type>transmission_interface/SimpleTransmission</type>
-    <joint name="${arm_id}_joint4">
-      <hardwareInterface>hardware_interface/PositionJointInterface</hardwareInterface>
-    </joint>
-    <actuator name="${arm_id}_joint4_motor">
-      <mechanicalReduction>1</mechanicalReduction>
-    </actuator>
-  </transmission>
-  <transmission name="${arm_id}_joint5_trans">
-    <type>transmission_interface/SimpleTransmission</type>
-    <joint name="${arm_id}_joint5">
-      <hardwareInterface>hardware_interface/PositionJointInterface</hardwareInterface>
-    </joint>
-    <actuator name="${arm_id}_joint5_motor">
-      <mechanicalReduction>1</mechanicalReduction>
-    </actuator>
-  </transmission>
-  <transmission name="${arm_id}_joint6_trans">
-    <type>transmission_interface/SimpleTransmission</type>
-    <joint name="${arm_id}_joint6">
-      <hardwareInterface>hardware_interface/PositionJointInterface</hardwareInterface>
-    </joint>
-    <actuator name="${arm_id}_joint6_motor">
-      <mechanicalReduction>1</mechanicalReduction>
-    </actuator>
-  </transmission>
-  <transmission name="${arm_id}_joint7_trans">
-    <type>transmission_interface/SimpleTransmission</type>
-    <joint name="${arm_id}_joint7">
-      <hardwareInterface>hardware_interface/PositionJointInterface</hardwareInterface>
-    </joint>
-    <actuator name="${arm_id}_joint7_motor">
+	<gazebo reference="panda_left_link0">
+      <material>Gazebo/Grey</material>
+          <mu1>0.2</mu1>
+          <mu2>0.2</mu2>
+  </gazebo>
+	<gazebo reference="panda_left_link1">
+      <material>Gazebo/Grey</material>
+          <mu1>0.2</mu1>
+          <mu2>0.2</mu2>
+  </gazebo>
+	<gazebo reference="panda_left_link2">
+      <material>Gazebo/Grey</material>
+          <mu1>0.2</mu1>
+          <mu2>0.2</mu2>
+  </gazebo>
+	<gazebo reference="panda_left_link3">
+      <material>Gazebo/Grey</material>
+          <mu1>0.2</mu1>
+          <mu2>0.2</mu2>
+  </gazebo>
+	<gazebo reference="panda_left_link4">
+      <material>Gazebo/Grey</material>
+          <mu1>0.2</mu1>
+          <mu2>0.2</mu2>
+  </gazebo>
+	<gazebo reference="panda_left_link5">
+      <material>Gazebo/Grey</material>
+          <mu1>0.2</mu1>
+          <mu2>0.2</mu2>
+  </gazebo>
+	<gazebo reference="panda_left_link6">
+      <material>Gazebo/Grey</material>
+          <mu1>0.2</mu1>
+          <mu2>0.2</mu2>
+  </gazebo>
+	<gazebo reference="panda_left_link7">
+      <material>Gazebo/Grey</material>
+          <mu1>0.2</mu1>
+          <mu2>0.2</mu2>
+  </gazebo>
+	<gazebo reference="panda_left_link8">
+      <material>Gazebo/Grey</material>
+          <mu1>0.2</mu1>
+          <mu2>0.2</mu2>
+  </gazebo>
+  <gazebo reference="panda_right_link0">
+      <material>Gazebo/Grey</material>
+          <mu1>0.2</mu1>
+          <mu2>0.2</mu2>
+  </gazebo>
+  <gazebo reference="panda_right_link1">
+      <material>Gazebo/Grey</material>
+          <mu1>0.2</mu1>
+          <mu2>0.2</mu2>
+  </gazebo>
+  <gazebo reference="panda_right_link2">
+      <material>Gazebo/Grey</material>
+          <mu1>0.2</mu1>
+          <mu2>0.2</mu2>
+  </gazebo>
+  <gazebo reference="panda_right_link3">
+      <material>Gazebo/Grey</material>
+          <mu1>0.2</mu1>
+          <mu2>0.2</mu2>
+  </gazebo>
+  <gazebo reference="panda_right_link4">
+      <material>Gazebo/Grey</material>
+          <mu1>0.2</mu1>
+          <mu2>0.2</mu2>
+  </gazebo>
+  <gazebo reference="panda_right_link5">
+      <material>Gazebo/Grey</material>
+          <mu1>0.2</mu1>
+          <mu2>0.2</mu2>
+  </gazebo>
+  <gazebo reference="panda_right_link6">
+      <material>Gazebo/Grey</material>
+          <mu1>0.2</mu1>
+          <mu2>0.2</mu2>
+  </gazebo>
+  <gazebo reference="panda_right_link7">
+      <material>Gazebo/Grey</material>
+          <mu1>0.2</mu1>
+          <mu2>0.2</mu2>
+  </gazebo>
+  <gazebo reference="panda_right_link8">
+      <material>Gazebo/Grey</material>
+          <mu1>0.2</mu1>
+          <mu2>0.2</mu2>
+  </gazebo>
+	 <transmission name="panda_left_joint1_trans">
+    <type>transmission_interface/SimpleTransmission</type>
+    <joint name="panda_left_joint1">
+      <hardwareInterface>hardware_interface/PositionJointInterface</hardwareInterface>
+    </joint>
+    <actuator name="panda_left_joint1_motor">
+      <mechanicalReduction>1</mechanicalReduction>
+    </actuator>
+  </transmission>
+  <transmission name="panda_right_joint1_trans">
+    <type>transmission_interface/SimpleTransmission</type>
+    <joint name="panda_right_joint1">
+      <hardwareInterface>hardware_interface/PositionJointInterface</hardwareInterface>
+    </joint>
+    <actuator name="panda_right_joint1_motor">
+      <mechanicalReduction>1</mechanicalReduction>
+    </actuator>
+  </transmission>
+  <transmission name="panda_left_joint2_trans">
+    <type>transmission_interface/SimpleTransmission</type>
+    <joint name="panda_left_joint2">
+      <hardwareInterface>hardware_interface/PositionJointInterface</hardwareInterface>
+    </joint>
+    <actuator name="panda_left_joint2_motor">
+      <mechanicalReduction>1</mechanicalReduction>
+    </actuator>
+  </transmission>
+  <transmission name="panda_right_joint2_trans">
+    <type>transmission_interface/SimpleTransmission</type>
+    <joint name="panda_right_joint2">
+      <hardwareInterface>hardware_interface/PositionJointInterface</hardwareInterface>
+    </joint>
+    <actuator name="panda_right_joint2_motor">
+      <mechanicalReduction>1</mechanicalReduction>
+    </actuator>
+  </transmission>
+  <transmission name="panda_left_joint3_trans">
+    <type>transmission_interface/SimpleTransmission</type>
+    <joint name="panda_left_joint3">
+      <hardwareInterface>hardware_interface/PositionJointInterface</hardwareInterface>
+    </joint>
+    <actuator name="panda_left_joint3_motor">
+      <mechanicalReduction>1</mechanicalReduction>
+    </actuator>
+  </transmission>
+  <transmission name="panda_right_joint3_trans">
+    <type>transmission_interface/SimpleTransmission</type>
+    <joint name="panda_right_joint3">
+      <hardwareInterface>hardware_interface/PositionJointInterface</hardwareInterface>
+    </joint>
+    <actuator name="panda_right_joint3_motor">
+      <mechanicalReduction>1</mechanicalReduction>
+    </actuator>
+  </transmission>
+  <transmission name="panda_left_joint4_trans">
+    <type>transmission_interface/SimpleTransmission</type>
+    <joint name="panda_left_joint4">
+      <hardwareInterface>hardware_interface/PositionJointInterface</hardwareInterface>
+    </joint>
+    <actuator name="panda_left_joint4_motor">
+      <mechanicalReduction>1</mechanicalReduction>
+    </actuator>
+  </transmission>
+  <transmission name="panda_right_joint4_trans">
+    <type>transmission_interface/SimpleTransmission</type>
+    <joint name="panda_right_joint4">
+      <hardwareInterface>hardware_interface/PositionJointInterface</hardwareInterface>
+    </joint>
+    <actuator name="panda_right_joint4_motor">
+      <mechanicalReduction>1</mechanicalReduction>
+    </actuator>
+  </transmission>
+  <transmission name="panda_left_joint5_trans">
+    <type>transmission_interface/SimpleTransmission</type>
+    <joint name="panda_left_joint5">
+      <hardwareInterface>hardware_interface/PositionJointInterface</hardwareInterface>
+    </joint>
+    <actuator name="panda_left_joint5_motor">
+      <mechanicalReduction>1</mechanicalReduction>
+    </actuator>
+  </transmission>
+  <transmission name="panda_right_joint5_trans">
+    <type>transmission_interface/SimpleTransmission</type>
+    <joint name="panda_right_joint5">
+      <hardwareInterface>hardware_interface/PositionJointInterface</hardwareInterface>
+    </joint>
+    <actuator name="panda_right_joint5_motor">
+      <mechanicalReduction>1</mechanicalReduction>
+    </actuator>
+  </transmission>
+  <transmission name="panda_left_joint6_trans">
+    <type>transmission_interface/SimpleTransmission</type>
+    <joint name="panda_left_joint6">
+      <hardwareInterface>hardware_interface/PositionJointInterface</hardwareInterface>
+    </joint>
+    <actuator name="panda_left_joint6_motor">
+      <mechanicalReduction>1</mechanicalReduction>
+    </actuator>
+  </transmission>
+  <transmission name="panda_right_joint6_trans">
+    <type>transmission_interface/SimpleTransmission</type>
+    <joint name="panda_right_joint6">
+      <hardwareInterface>hardware_interface/PositionJointInterface</hardwareInterface>
+    </joint>
+    <actuator name="panda_right_joint6_motor">
+      <mechanicalReduction>1</mechanicalReduction>
+    </actuator>
+  </transmission>
+  <transmission name="panda_left_joint7_trans">
+    <type>transmission_interface/SimpleTransmission</type>
+    <joint name="panda_left_joint7">
+      <hardwareInterface>hardware_interface/PositionJointInterface</hardwareInterface>
+    </joint>
+    <actuator name="panda_left_joint7_motor">
+      <mechanicalReduction>1</mechanicalReduction>
+    </actuator>
+  </transmission>
+  <transmission name="panda_right_joint7_trans">
+    <type>transmission_interface/SimpleTransmission</type>
+    <joint name="panda_right_joint7">
+      <hardwareInterface>hardware_interface/PositionJointInterface</hardwareInterface>
+    </joint>
+    <actuator name="panda_right_joint7_motor">
       <mechanicalReduction>1</mechanicalReduction>
     </actuator>
