Commit message: new dual arm formulation

File: franka_gazebo/robots/panda_arm.xacro (robot description, xacro)
@@ -1,7 +1,6 @@
 <?xml version='1.0' encoding='utf-8'?>
 <robot xmlns:xacro="http://www.ros.org/wiki/xacro" name="panda">
-  <xacro:macro name="panda_arm" params="arm_id:='panda' package_name:='franka_gazebo' connected_to:=''  xyz:='0 0 0' rpy:='0 0 0'">
+  <xacro:macro name="panda_arm" params="arm_id:='panda' description_pkg:='franka_gazebo' connected_to:='' xyz:='0 0 0' rpy:='0 0 0' safety_distance:=0">
     <xacro:unless value="${not connected_to}">
-      <link name="${connected_to}"/>
       <joint name="${arm_id}_joint_${connected_to}" type="fixed">
         <parent link="${connected_to}"/>
@@ -10,49 +9,80 @@
       </joint>
     </xacro:unless>
-    <xacro:arg name="gazebo" default="true"/>
-    <xacro:if value="$(arg gazebo)">
-      <!-- Gazebo Tags -->
-      <xacro:include filename="$(find franka_gazebo)/robots/panda_arm.gazebo.xacro"/>
+    <xacro:property name="joint_damping" value="1.0"/>
+    <!--xacro:arg name="gazebo" default="true"/>
+    <xacro:arg name="gazu" default="panda_left"/>
+    <xacro:property name="var" value="${arm_id}"/-->
+    <!--xacro:include filename="$(find franka_gazebo)/robots/panda_arm.gazebo.xacro"/-->
+    <!--xacro:if value="${(var == 'panda_left') }">
+      <xacro:include filename="$(find franka_gazebo)/robots/panda_arm.gazebo_left.xacro"/>
     </xacro:if>
-    <link name="${arm_id}_link0">
-      <inertial>
-        <mass value="2.92" />
-        <origin xyz="-0.025566 -2.88e-05 0.057332" rpy="0 0 0" />
-        <inertia ixx="0.00782229414331" ixy="-1.56191622996e-05" ixz="-0.00126005738123" iyy="0.0109027971813" iyz="1.08233858202e-05" izz="0.0102355503949" />
-      </inertial>
-      <visual>
-        <origin xyz="${xyz}" rpy="${rpy}"/>
-        <geometry>
-          <mesh filename="package://${package_name}/meshes/visual/link0.dae"/>
-        </geometry>
-      </visual>
-      <collision>
-        <origin xyz="${xyz}" rpy="${rpy}"/>
-        <geometry>
-          <mesh filename="package://${package_name}/meshes/collision/link0.stl"/>
-        </geometry>
-      </collision>
+    <xacro:if value="${(var == 'panda_right') }">
+      <xacro:include filename="$(find franka_gazebo)/robots/panda_arm.gazebo_right.xacro"/>
+    </xacro:if-->
+    <!--xacro:if value="${var == 'panda_left'}"/-->
+      <!--xacro:include filename="$(find franka_gazebo)/robots/panda_arm.gazebo_left.xacro"/-->
+    <!--/xacro:if-->
+    <!--xacro:if value="${var == 'panda_right'}"/>
+      <xacro:include filename="$(find franka_gazebo)/robots/panda_arm.gazebo_right.xacro"/>
+    </xacro:if-->
+   <link name="${arm_id}_link0">
+      <visual>
+        <geometry>
+          <mesh filename="package://${description_pkg}/meshes/visual/link0.dae"/>
+        </geometry>
+      </visual>
+      <collision>
+        <origin xyz="-0.075 0 0.06" rpy="0 ${pi/2} 0"/>
+        <geometry>
+          <cylinder radius="${0.06+safety_distance}" length="0.03" />
+        </geometry>
+      </collision>
+      <collision>
+        <origin xyz="-0.06 0 0.06" rpy="0 0 0"/>
+        <geometry>
+          <sphere radius="${0.06+safety_distance}" />
+        </geometry>
+      </collision>
+      <collision>
+        <origin xyz="-0.09 0 0.06" rpy="0 0 0"/>
+        <geometry>
+          <sphere radius="${0.06+safety_distance}" />
+        </geometry>
+      </collision>
+      <inertial>
+        <origin xyz="0 0 0" rpy="0 0 0"/>
+        <mass value="3.06"/>
+        <inertia ixx="0.3" ixy="0.0" ixz="0.0" iyy="0.3" iyz="0.0" izz="0.3"/>
+      </inertial>
     </link>
     <link name="${arm_id}_link1">
-      <inertial>
-        <mass value="2.74" />
-        <origin xyz="0 -0.0324958 -0.0675818" rpy="0 0 0" />
-        <inertia ixx="0.0180416958283" ixy="0.0" ixz="0.0" iyy="0.0159136071891" iyz="0.0046758424612" izz="0.00620690827127" />
-      </inertial>
-      <visual>
-        <origin xyz="${xyz}" rpy="${rpy}"/>
-        <geometry>
-          <mesh filename="package://${package_name}/meshes/visual/link1.dae"/>
-        </geometry>
-        <material name="">
-          <color rgba="1 1 1 1"/>
-        </material>
-      </visual>
-      <collision>
-        <origin xyz="${xyz}" rpy="${rpy}"/>
-        <geometry>
-          <mesh filename="package://${package_name}/meshes/collision/link1.stl"/>
-        </geometry>
-      </collision>
+      <visual>
+        <geometry>
+          <mesh filename="package://${description_pkg}/meshes/visual/link1.dae"/>
+        </geometry>
+      </visual>
+      <collision>
+        <origin xyz="0 0 -0.1915" rpy="0 0 0"/>
+        <geometry>
+          <cylinder radius="${0.06+safety_distance}" length="0.2830" />
+        </geometry>
+      </collision>
+      <collision>
+        <origin xyz="0 0 -0.333" rpy="0 0 0"/>
+        <geometry>
+          <sphere radius="${0.06+safety_distance}" />
+        </geometry>
+      </collision>
+      <collision>
+        <origin xyz="0 0 -0.05" rpy="0 0 0"/>
+        <geometry>
+          <sphere radius="${0.06+safety_distance}" />
+        </geometry>
+      </collision>
+      <inertial>
+        <origin xyz="0 0 0" rpy="0 0 0"/>
+        <mass value="2.34"/>
+        <inertia ixx="0.3" ixy="0.0" ixz="0.0" iyy="0.3" iyz="0.0" izz="0.3"/>
+      </inertial>
     </link>
     <joint name="${arm_id}_joint1" type="revolute">
@@ -63,26 +93,35 @@
       <axis xyz="0 0 1"/>
       <limit effort="87" lower="-2.8973" upper="2.8973" velocity="2.1750"/>
+      <dynamics damping="${joint_damping}"/>
     </joint>
     <link name="${arm_id}_link2">
-      <inertial>
-        <mass value="2.74" />
-        <origin xyz="0 -0.06861 0.0322285" rpy="0 0 0" />
-        <inertia ixx="0.0182856182281" ixy="0.0" ixz="0.0" iyy="0.00621358421175" iyz="-0.00472844221905" izz="0.0161514346309" />
-      </inertial>
-      <visual>
-        <origin xyz="${xyz}" rpy="${rpy}"/>
-        <geometry>
-          <mesh filename="package://${package_name}/meshes/visual/link2.dae"/>
-        </geometry>
-        <material name="">
-          <color rgba="1 1 1 1"/>
-        </material>
-      </visual>
-      <collision>
-        <origin xyz="${xyz}" rpy="${rpy}"/>
-        <geometry>
-          <mesh filename="package://${package_name}/meshes/collision/link2.stl"/>
-        </geometry>
-      </collision>
+      <visual>
+        <geometry>
+          <mesh filename="package://${description_pkg}/meshes/visual/link2.dae"/>
+        </geometry>
+      </visual>
+      <collision>
+        <origin xyz="0 0 0" rpy="0 0 0"/>
+        <geometry>
+          <cylinder radius="${0.06+safety_distance}" length="0.12" />
+        </geometry>
+      </collision>
+      <collision>
+        <origin xyz="0 0 -0.06" rpy="0 0 0"/>
+        <geometry>
+          <sphere radius="${0.06+safety_distance}" />
+        </geometry>
+      </collision>
+      <collision>
+        <origin xyz="0 0 0.06" rpy="0 0 0"/>
+        <geometry>
+          <sphere radius="${0.06+safety_distance}" />
+        </geometry>
+      </collision>
+      <inertial>
+        <origin xyz="0 0 0" rpy="0 0 0"/>
+        <mass value="2.36"/>
+        <inertia ixx="0.3" ixy="0.0" ixz="0.0" iyy="0.3" iyz="0.0" izz="0.3"/>
+      </inertial>
     </link>
     <joint name="${arm_id}_joint2" type="revolute">
@@ -95,24 +134,32 @@
     </joint>
     <link name="${arm_id}_link3">
-      <inertial>
-        <mass value="2.38" />
-        <origin xyz="0.0469893 0.0316374 -0.031704" rpy="0 0 0" />
-        <inertia ixx="0.00771376630908" ixy="-0.00248490625138" ixz="-0.00332147581033" iyy="0.00989108008727" iyz="-0.00217796151484" izz="0.00811723558464" />
-      </inertial>
-      <visual>
-        <origin xyz="${xyz}" rpy="${rpy}"/>
-        <geometry>
-          <mesh filename="package://${package_name}/meshes/visual/link3.dae"/>
-        </geometry>
-        <material name="">
-          <color rgba="1 1 1 1"/>
-        </material>
-      </visual>
-      <collision>
-        <origin xyz="${xyz}" rpy="${rpy}"/>
-        <geometry>
-          <mesh filename="package://${package_name}/meshes/collision/link3.stl"/>
-        </geometry>
-      </collision>
+      <visual>
+        <geometry>
+          <mesh filename="package://${description_pkg}/meshes/visual/link3.dae"/>
+        </geometry>
+      </visual>
+      <collision>
+        <origin xyz="0 0 -0.145" rpy="0 0 0"/>
+        <geometry>
+          <cylinder radius="${0.06+safety_distance}" length="0.15" />
+        </geometry>
+      </collision>
+      <collision>
+        <origin xyz="0 0 -0.22" rpy="0 0 0"/>
+        <geometry>
+          <sphere radius="${0.06+safety_distance}" />
+        </geometry>
+      </collision>
+      <collision>
+        <origin xyz="0 0 -0.07" rpy="0 0 0"/>
+        <geometry>
+          <sphere radius="${0.06+safety_distance}" />
+        </geometry>
+      </collision>
+      <inertial>
+        <origin xyz="0 0 0" rpy="0 0 0"/>
+        <mass value="2.38"/>
+        <inertia ixx="0.3" ixy="0.0" ixz="0.0" iyy="0.3" iyz="0.0" izz="0.3"/>
+      </inertial>
     </link>
     <joint name="${arm_id}_joint3" type="revolute">
@@ -125,56 +172,88 @@
     </joint>
     <link name="${arm_id}_link4">
-      <inertial>
-        <mass value="2.38" />
-        <origin xyz="-0.0360446 0.0336853 0.031882" rpy="0 0 0" />
-        <inertia ixx="0.00799663881132" ixy="0.00347095570217" ixz="-0.00241222942995" iyy="0.00825390705278" iyz="0.00235774044121" izz="0.0102515004345" />
-      </inertial>
-      <visual>
-        <origin xyz="${xyz}" rpy="${rpy}"/>
-        <geometry>
-          <mesh filename="package://${package_name}/meshes/visual/link4.dae"/>
-        </geometry>
-        <material name="">
-          <color rgba="1 1 1 1"/>
-        </material>
-      </visual>
-      <collision>
-        <origin xyz="${xyz}" rpy="${rpy}"/>
-        <geometry>
-          <mesh filename="package://${package_name}/meshes/collision/link4.stl"/>
-        </geometry>
-      </collision>
+      <visual>
+        <geometry>
+          <mesh filename="package://${description_pkg}/meshes/visual/link4.dae"/>
+        </geometry>
+      </visual>
+      <collision>
+        <origin xyz="0 0 0" rpy="0 0 0"/>
+        <geometry>
+          <cylinder radius="${0.06+safety_distance}" length="0.12" />
+        </geometry>
+      </collision>
+      <collision>
+        <origin xyz="0 0 0.06" rpy="0 0 0"/>
+        <geometry>
+          <sphere radius="${0.06+safety_distance}" />
+        </geometry>
+      </collision>
+      <collision>
+        <origin xyz="0 0 -0.06" rpy="0 0 0"/>
+        <geometry>
+          <sphere radius="${0.06+safety_distance}" />
+        </geometry>
+      </collision>
+      <inertial>
+        <origin xyz="0 0 0" rpy="0 0 0"/>
+        <mass value="2.43"/>
+        <inertia ixx="0.3" ixy="0.0" ixz="0.0" iyy="0.3" iyz="0.0" izz="0.3"/>
+      </inertial>
     </link>
     <joint name="${arm_id}_joint4" type="revolute">
-      <safety_controller k_position="100.0" k_velocity="40.0" soft_lower_limit="-3.0718" soft_upper_limit="0.0698"/>
-      <!-- soft_upper_limitr should be -0.0698, but that brakes simulation when initial position for this joint is 0.0 -->
+      <safety_controller k_position="100.0" k_velocity="40.0" soft_lower_limit="-3.0718" soft_upper_limit="-0.0698"/>
       <origin rpy="${pi/2} 0 0" xyz="0.0825 0 0"/>
       <parent link="${arm_id}_link3"/>
       <child link="${arm_id}_link4"/>
       <axis xyz="0 0 1"/>
-      <limit effort="87" lower="-3.0718" upper="0.0698" velocity="2.1750"/>
-      <!-- upper should be -0.0698, but that brakes simulation when initial position for this joint is 0.0 -->
+      <limit effort="87" lower="-3.0718" upper="-0.0698" velocity="2.1750"/>
     </joint>
     <link name="${arm_id}_link5">
-      <inertial>
-        <mass value="2.74" />
-        <origin xyz="0 0.0610427 -0.104176" rpy="0 0 0" />
-        <inertia ixx="0.030371374513" ixy="6.50283587108e-07" ixz="-1.05129179916e-05" iyy="0.0288752887402" iyz="-0.00775653445787" izz="0.00444134056164" />
-      </inertial>
-      <visual>
-        <origin xyz="${xyz}" rpy="${rpy}"/>
-        <geometry>
-          <mesh filename="package://${package_name}/meshes/visual/link5.dae"/>
-        </geometry>
-        <material name="">
-          <color rgba="1 1 1 1"/>
-        </material>
-      </visual>
-      <collision>
-        <origin xyz="${xyz}" rpy="${rpy}"/>
-        <geometry>
-          <mesh filename="package://${package_name}/meshes/collision/link5.stl"/>
-        </geometry>
-      </collision>
+      <visual>
+        <geometry>
+          <mesh filename="package://${description_pkg}/meshes/visual/link5.dae"/>
+        </geometry>
+      </visual>
+      <collision>
+        <origin xyz="0 0 -0.26" rpy="0 0 0"/>
+        <geometry>
+          <cylinder radius="${0.06+safety_distance}" length="0.1" />
+        </geometry>
+      </collision>
+      <collision>
+        <origin xyz="0 0 -0.31" rpy="0 0 0"/>
+        <geometry>
+          <sphere radius="${0.06+safety_distance}" />
+        </geometry>
+      </collision>
+      <collision>
+        <origin xyz="0 0 -0.21" rpy="0 0 0"/>
+        <geometry>
+          <sphere radius="${0.06+safety_distance}" />
+        </geometry>
+      </collision>
+      <collision>
+        <origin xyz="0 0.08 -0.13" rpy="0 0 0"/>
+        <geometry>
+          <cylinder radius="${0.025+safety_distance}" length="0.14" />
+        </geometry>
+      </collision>
+      <collision>
+        <origin xyz="0 0.08 -0.06" rpy="0 0 0"/>
+        <geometry>
+          <sphere radius="${0.025+safety_distance}" />
+        </geometry>
+      </collision>
+      <collision>
+        <origin xyz="0 0.08 -0.20" rpy="0 0 0"/>
+        <geometry>
+          <sphere radius="${0.025+safety_distance}" />
+        </geometry>
+      </collision>
+      <inertial>
+        <origin xyz="0 0 0" rpy="0 0 0"/>
+        <mass value="3.5"/>
+        <inertia ixx="0.3" ixy="0.0" ixz="0.0" iyy="0.3" iyz="0.0" izz="0.3"/>
+      </inertial>
     </link>
     <joint name="${arm_id}_joint5" type="revolute">
@@ -187,24 +266,32 @@
     </joint>
     <link name="${arm_id}_link6">
-      <inertial>
-        <mass value="1.55" />
-        <origin xyz="0.0510509 0.009108 0.0106343" rpy="0 0 0" />
-        <inertia ixx="0.00303336450376" ixy="-0.000437276865508" ixz="0.000629257294877" iyy="0.00404479911567" iyz="0.000130472021025" izz="0.00558234286039" />
-      </inertial>
-      <visual>
-        <origin xyz="${xyz}" rpy="${rpy}"/>
-        <geometry>
-          <mesh filename="package://${package_name}/meshes/visual/link6.dae"/>
-        </geometry>
-        <material name="">
-          <color rgba="1 1 1 1"/>
-        </material>
-      </visual>
-      <collision>
-        <origin xyz="${xyz}" rpy="${rpy}"/>
-        <geometry>
-          <mesh filename="package://${package_name}/meshes/collision/link6.stl"/>
-        </geometry>
-      </collision>
+      <visual>
+        <geometry>
+          <mesh filename="package://${description_pkg}/meshes/visual/link6.dae"/>
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